Commit message: 260709 update latest description files

File: urdf/MagicBotZ1.urdf (robot description, URDF)
Before this commit: robot MagicBotZ1, 31 links, 30 joints
Links:
- removed link LINK_ANKLE_PITCH_L
- removed link LINK_ANKLE_PITCH_R
- removed link LINK_ANKLE_ROLL_L
- removed link LINK_ANKLE_ROLL_R
- removed link LINK_FOOT_L
- removed link LINK_FOOT_R
- removed link LINK_HAND_L
- removed link LINK_HAND_R
- removed link LINK_HIP_PITCH_L
- removed link LINK_HIP_PITCH_R
- removed link LINK_HIP_ROLL_L
- removed link LINK_HIP_ROLL_R
- removed link LINK_HIP_YAW_L
- removed link LINK_HIP_YAW_R
- removed link LINK_KNEE_PITCH_L
- removed link LINK_KNEE_PITCH_R
- removed link LINK_TOE_L
- removed link LINK_TOE_R
- removed link link_hy
- removed link link_la1
- removed link link_la2
- removed link link_la3
- removed link link_la4
- removed link link_la5
- removed link link_ra1
- removed link link_ra2
- removed link link_ra3
- removed link link_ra4
- removed link link_ra5
- removed link link_wy
- added link head_link, mass 0.7987; collision mesh filename=package://magicbot-z1_description/meshes/head_link.STL; visual mesh filename=package://magicbot-z1_description/meshes/head_link.STL
- added link left_ankle_pitch_link, mass 0.048544; collision mesh filename=package://magicbot-z1_description/meshes/left_ankle_pitch_l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; visual mesh filename=package://magicbot-z1_description/meshes/left_ankle_pitch_l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
- added link left_ankle_roll_link, mass 0.7019; collision mesh filename=package://magicbot-z1_description/meshes/left_ankle_roll_li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; visual mesh filename=package://magicbot-z1_description/meshes/left_ankle_roll_li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
- added link left_elbow_link, mass 1.48; collision mesh filename=package://magicbot-z1_description/meshes/left_elbow_link.STL; visual mesh filename=package://magicbot-z1_description/meshes/left_elbow_link.STL
- added link left_hand_palm_link, mass 1e-12; collision cylinder length=0.075 radius=0.0225
- added link left_hip_pitch_link, mass 1.5089; collision mesh filename=package://magicbot-z1_description/meshes/left_hip_pitch_lin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; visual mesh filename=package://magicbot-z1_description/meshes/left_hip_pitch_lin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
- added link left_hip_roll_link, mass 1.9215; collision mesh filename=package://magicbot-z1_description/meshes/left_hip_roll_link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; visual mesh filename=package://magicbot-z1_description/meshes/left_hip_roll_link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
- added link left_hip_yaw_link, mass 0.9002; collision mesh filename=package://magicbot-z1_description/meshes/left_hip_yaw_link.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; visual mesh filename=package://magicbot-z1_description/meshes/left_hip_yaw_link.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
- added link left_knee_link, mass 3.7275; collision mesh filename=package://magicbot-z1_description/meshes/left_knee_link.STL; visual mesh filename=package://magicbot-z1_description/meshes/left_knee_link.STL
- added link left_shoulder_pitch_link, mass 0.8939; collision mesh filename=package://magicbot-z1_description/meshes/left_shoulder_pitc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; visual mesh filename=package://magicbot-z1_description/meshes/left_shoulder_pitc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
- added link left_shoulder_roll_link, mass 0.7787; collision cylinder length=0.05 radius=0.032; visual mesh filename=package://magicbot-z1_description/meshes/left_shoulder_roll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
- added link left_shoulder_yaw_link, mass 0.35928; collision mesh filename=package://magicbot-z1_description/meshes/left_shoulder_yaw_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; visual mesh filename=package://magicbot-z1_description/meshes/left_shoulder_yaw_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
- added link left_wrist_roll_link, mass 0.2728; collision cylinder length=0.085 radius=0.0275; visual mesh filename=package://magicbot-z1_description/meshes/left_wrist_yaw_lin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
- added link right_ankle_pitch_link, mass 0.048544; collision mesh filename=package://magicbot-z1_description/meshes/right_ankle_pitch_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; visual mesh filename=package://magicbot-z1_description/meshes/right_ankle_pitch_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
- added link right_ankle_roll_link, mass 0.70183; collision mesh filename=package://magicbot-z1_description/meshes/right_ankle_roll_l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; visual mesh filename=package://magicbot-z1_description/meshes/right_ankle_roll_l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
- added link right_elbow_link, mass 1.48; collision mesh filename=package://magicbot-z1_description/meshes/right_elbow_link.S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; visual mesh filename=package://magicbot-z1_description/meshes/right_elbow_link.S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
- added link right_hand_palm_link, mass 1e-12; collision cylinder length=0.075 radius=0.0225
- added link right_hip_pitch_link, mass 1.5089; collision mesh filename=package://magicbot-z1_description/meshes/right_hip_pitch_li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; visual mesh filename=package://magicbot-z1_description/meshes/right_hip_pitch_li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
- added link right_hip_roll_link, mass 1.9215; collision mesh filename=package://magicbot-z1_description/meshes/right_hip_roll_lin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; visual mesh filename=package://magicbot-z1_description/meshes/right_hip_roll_lin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
- added link right_hip_yaw_link, mass 0.9002; collision mesh filename=package://magicbot-z1_description/meshes/right_hip_yaw_link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; visual mesh filename=package://magicbot-z1_description/meshes/right_hip_yaw_link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
- added link right_knee_link, mass 3.7292; collision mesh filename=package://magicbot-z1_description/meshes/right_knee_link.STL; visual mesh filename=package://magicbot-z1_description/meshes/right_knee_link.STL
- added link right_shoulder_pitch_link, mass 0.8976; collision mesh filename=package://magicbot-z1_description/meshes/right_shoulder_pit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; visual mesh filename=package://magicbot-z1_description/meshes/right_shoulder_pit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
- added link right_shoulder_roll_link, mass 0.7868; collision cylinder length=0.05 radius=0.032; visual mesh filename=package://magicbot-z1_description/meshes/right_shoulder_rol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
- added link right_shoulder_yaw_link, mass 0.3593; collision mesh filename=package://magicbot-z1_description/meshes/right_shoulder_yaw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; visual mesh filename=package://magicbot-z1_description/meshes/right_shoulder_yaw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
- added link right_wrist_roll_link, mass 0.27279; collision cylinder length=0.085 radius=0.0275; visual mesh filename=package://magicbot-z1_description/meshes/right_wrist_yaw_li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
- added link torso_link, mass 9.8779; collision mesh filename=package://magicbot-z1_description/meshes/torso_link.STL; visual mesh filename=package://magicbot-z1_description/meshes/torso_link.STL
- link pelvis: geometry collision sphere radius=0.065; visual mesh filename=package://magicbot-z1_description/meshes/pelvis.STL
Joints:
- removed joint JOINT_ANKLE_PITCH_L
- removed joint JOINT_ANKLE_PITCH_R
- removed joint JOINT_ANKLE_ROLL_L
- removed joint JOINT_ANKLE_ROLL_R
- removed joint JOINT_HIP_PITCH_L
- removed joint JOINT_HIP_PITCH_R
- removed joint JOINT_HIP_ROLL_L
- removed joint JOINT_HIP_ROLL_R
- removed joint JOINT_HIP_YAW_L
- removed joint JOINT_HIP_YAW_R
- removed joint JOINT_KNEE_PITCH_L
- removed joint JOINT_KNEE_PITCH_R
- removed joint JOINT_TOE_L
- removed joint JOINT_TOE_R
- removed joint J_FOOT_L
- removed joint J_FOOT_R
- removed joint J_HAND_L
- removed joint J_HAND_R
- removed joint joint_hy
- removed joint joint_la1
- removed joint joint_la2
- removed joint joint_la3
- removed joint joint_la4
- removed joint joint_la5
- removed joint joint_ra1
- removed joint joint_ra2
- removed joint joint_ra3
- removed joint joint_ra4
- removed joint joint_ra5
- removed joint joint_wy
- added joint head_joint: type fixed, parent torso_link, child head_link, origin xyz=0 0 0.4889 rpy=0 0 0, axis 0 0 1, limit lower=-0.6981 upper=0.6981 effort=50 velocity=18
- added joint left_ankle_pitch_joint: type revolute, parent left_knee_link, child left_ankle_pitch_link, origin xyz=0 0 -0.34 rpy=0 0 0, axis 0 1 0, limit lower=-0.873 upper=0.524 effort=50 velocity=18
- added joint left_ankle_roll_joint: type revolute, parent left_ankle_pitch_link, child left_ankle_roll_link, origin xyz=0 0 -0.018 rpy=0 0 0, axis 1 0 0, limit lower=-0.262 upper=0.262 effort=50 velocity=18
- added joint left_elbow_joint: type revolute, parent left_shoulder_yaw_link, child left_elbow_link, origin xyz=0.01924 0 -0.0979 rpy=0 0 0, axis 0 1 0, limit lower=-0.96 upper=2.0944 effort=50 velocity=18
- added joint left_hand_palm_joint: type fixed, parent left_wrist_roll_link, child left_hand_palm_link, origin xyz=0.129 0.000000 -0. rpy=0 0 0, axis 0 0 1
- added joint left_hip_pitch_joint: type revolute, parent pelvis, child left_hip_pitch_link, origin xyz=0 0.06875 0 rpy=0 0 0, axis 0 1 0, limit lower=-2.7925 upper=2.7925 effort=120 velocity=35
- added joint left_hip_roll_joint: type revolute, parent left_hip_pitch_link, child left_hip_roll_link, origin xyz=0 0.053724 -0.045579 rpy=0 0 0, axis 1 0 0, limit lower=-0.524 upper=2.967 effort=120 velocity=35
- added joint left_hip_yaw_joint: type revolute, parent left_hip_roll_link, child left_hip_yaw_link, origin xyz=-0.00084052 0 -0.1255 rpy=0 0 0, axis 0 0 1, limit lower=-2.7925 upper=2.7925 effort=120 velocity=35
- added joint left_knee_joint: type revolute, parent left_hip_yaw_link, child left_knee_link, origin xyz=-0.052111 0 -0.13729 rpy=0 0 0, axis 0 1 0, limit lower=0 upper=2.653 effort=120 velocity=35
- added joint left_shoulder_pitch_joint: type revolute, parent torso_link, child left_shoulder_pitch_link, origin xyz=0 0.11963 0.3208 rpy=0.122173 0 0, axis 0 1 0, limit lower=-2.88 upper=2.88 effort=50 velocity=18
- added joint left_shoulder_roll_joint: type revolute, parent left_shoulder_pitch_link, child left_shoulder_roll_link, origin xyz=0 0.047187 -0.013786 rpy=-0.122173 0 0, axis 1 0 0, limit lower=-0.175 upper=2.2515 effort=50 velocity=18
- added joint left_shoulder_yaw_joint: type revolute, parent left_shoulder_roll_link, child left_shoulder_yaw_link, origin xyz=0 0 -0.1171 rpy=0 0 0, axis 0 0 1, limit lower=-2.618 upper=2.618 effort=50 velocity=18
- added joint left_wrist_roll_joint: type revolute, parent left_elbow_link, child left_wrist_roll_link, origin xyz=0.138 0 -0.017415 rpy=0 0 0, axis 1 0 0, limit lower=-2.618 upper=2.618 effort=50 velocity=18
- added joint right_ankle_pitch_joint: type revolute, parent right_knee_link, child right_ankle_pitch_link, origin xyz=0 0 -0.34 rpy=0 0 0, axis 0 1 0, limit lower=-0.873 upper=0.524 effort=50 velocity=18
- added joint right_ankle_roll_joint: type revolute, parent right_ankle_pitch_link, child right_ankle_roll_link, origin xyz=0 0 -0.018 rpy=0 0 0, axis 1 0 0, limit lower=-0.262 upper=0.262 effort=50 velocity=18
- added joint right_elbow_joint: type revolute, parent right_shoulder_yaw_link, child right_elbow_link, origin xyz=0.01924 0 -0.0979 rpy=0 0 0, axis 0 1 0, limit lower=-0.96 upper=2.0944 effort=50 velocity=18
- added joint right_hand_palm_joint: type fixed, parent right_wrist_roll_link, child right_hand_palm_link, origin xyz=0.129 0.000000 0.0 rpy=0 0 0, axis 0 0 1
- added joint right_hip_pitch_joint: type revolute, parent pelvis, child right_hip_pitch_link, origin xyz=0 -0.06875 0 rpy=0 0 0, axis 0 1 0, limit lower=-2.7925 upper=2.7925 effort=120 velocity=35
- added joint right_hip_roll_joint: type revolute, parent right_hip_pitch_link, child right_hip_roll_link, origin xyz=0 -0.053724 -0.045579 rpy=0 0 0, axis 1 0 0, limit lower=-2.967 upper=0.524 effort=120 velocity=35
- added joint right_hip_yaw_joint: type revolute, parent right_hip_roll_link, child right_hip_yaw_link, origin xyz=-0.00050599 0.0029213 -0.12555 rpy=0 0 0, axis 0 0 1, limit lower=-2.7925 upper=2.7925 effort=120 velocity=35
- added joint right_knee_joint: type revolute, parent right_hip_yaw_link, child right_knee_link, origin xyz=-0.052111 0 -0.13729 rpy=0 0 0, axis 0 1 0, limit lower=0 upper=2.653 effort=120 velocity=35
- added joint right_shoulder_pitch_joint: type revolute, parent torso_link, child right_shoulder_pitch_link, origin xyz=0 -0.11963 0.3208 rpy=-0.122173 0 0, axis 0 1 0, limit lower=-2.88 upper=2.88 effort=50 velocity=18
- added joint right_shoulder_roll_joint: type revolute, parent right_shoulder_pitch_link, child right_shoulder_roll_link, origin xyz=0 -0.047187 -0.013786 rpy=0.122173 0 0, axis 1 0 0, limit lower=-2.2515 upper=0.175 effort=50 velocity=18
- added joint right_shoulder_yaw_joint: type revolute, parent right_shoulder_roll_link, child right_shoulder_yaw_link, origin xyz=0 0 -0.1171 rpy=0 0 0, axis 0 0 1, limit lower=-2.618 upper=2.618 effort=50 velocity=18
- added joint right_wrist_roll_joint: type revolute, parent right_elbow_link, child right_wrist_roll_link, origin xyz=0.138 0 -0.017415 rpy=0 0 0, axis 1 0 0, limit lower=-2.618 upper=2.618 effort=50 velocity=18
- added joint waist_yaw_joint: type revolute, parent pelvis, child torso_link, origin xyz=0 0 0.0619 rpy=0 0 0, axis 0 0 1, limit lower=-2.79 upper=2.79 effort=120 velocity=35
